Commit message: second-order sliding surface implementation (match with library)

File: src/usv_description/urdf/usv.urdf (robot description, URDF)
Before this commit: robot usv, 1 links, 0 joints
Links:
- link usv: mass 30.0 -> None; geometry visual mesh filename=package://usv_description/models/vtec_s3/meshes/vtec_s3.dae scale=.1 .1 .1

Commit message: changes

File: src/usv_description/urdf/usv.urdf (robot description, URDF)
Before this commit: robot usv, 1 links, 0 joints
Links:
- link usv: geometry visual mesh filename=package://usv_description/models/vtec_s4/meshes/vtec_s4.dae scale=1 1 1

Commit message: demo ready in rviz

File: src/usv_description/urdf/usv.urdf (robot description, URDF)
Before this commit: robot usv, 1 links, 0 joints
Links:
- link usv: geometry visual mesh filename=package://usv_description/models/vtec_s3/meshes/vtec_s3.dae scale=.1 .1 .1
