Commit message: can update

File: src/usv_description/urdf/vtecs4.urdf (robot description, URDF)
Before this commit: robot usv_comms/usv, 1 links, 0 joints
Links:
- removed link usv_comms/usv
- added link usv; visual mesh filename=package://usv_description/models/vtec_s4/meshes/vtec_s4.dae scale=1 1 1

Commit message: mpc uses real dynamics, listens to rviz's ui's goal pose, and reaches targets

File: src/usv_description/urdf/vtecs4.urdf (robot description, URDF)
Before this commit: robot usv, 1 links, 0 joints
Links:
- link usv: geometry visual mesh filename=package://usv_description/models/vtec_s4/meshes/usv.dae scale=1 1 1

Commit message: better dae model for gz and rviz

File: src/usv_description/urdf/vtecs4.urdf (robot description, URDF)
Before this commit: robot usv, 1 links, 0 joints
Links:
- link usv: geometry visual mesh filename=package://usv_description/models/vtec_s4/meshes/asv.dae scale=1 1 1
